Commit message: cleaner apartment

File: apartment_without_walls.urdf (robot description, URDF)
Before this commit: robot apartment, 102 links, 101 joints
Links:
- removed link armchair
- removed link bedside_table
- removed link coffee_table
- removed link coffee_table_drawer
- removed link sofa
- removed link table_area_main_temp_raytest_fix
- added link coffe_machine; collision box size=0.58 0.32 0.41; visual box size=0.58 0.33 0.41
Joints:
- removed joint armchair_joint
- removed joint bedside_table_joint
- removed joint coffee_table_drawer_joint
- removed joint coffee_table_joint
- removed joint sofa_joint
- removed joint table_area_main_temp_raytest_fix_joint
- added joint coffe_machine_joint: type fixed, parent countertop, child coffe_machine, origin xyz=0 0.3 0.2
- joint cabinet3_door_top_out_joint: limit lower=0.0 upper=0.02 effort=1.0 velocity=1.5708 -> lower=0.0 upper=1.5708 effort=1.0 velocity=1.5708; type prismatic -> revolute
